File: 4ch-spdt-relay-1fan-pcb.kicad_pcb (KiCad board)
At the start: 2 copper layers, 107.9 x 62.8 mm, 49 parts, among them J1 Screw_Terminal_01x03, J2 Conn_01x08_Pin, J3 Screw_Terminal_01x03, J4 Screw_Terminal_01x03, J5 Screw_Terminal_01x03, K1 G5LE-1, K2 G5LE-1, K3 G5LE-1, K4 G5LE-1, Q1 2N3904, Q2 2N3904, Q3 2N3904, Q4 2N3904, Q5 BT136, U5 MOC3021M, U6 PC817

Commit message: Add files via upload
Routing:
- net GND: track 126.5 -> 120.3 mm
Changed lines of the file:
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@@
 			(outputformat 4)
 			(mirror no)
-			(drillshape 0)
+			(drillshape 2)
 			(scaleselection 1)
 			(outputdirectory "")
@@
 	)
 	(segment
-		(start 170.31 71.16)
-		(end 171.105 71.955)
-		(width 1)
-		(layer "B.Cu")
-		(net "GND")
-	)
-	(segment
 		(start 117.79 77.56)
 		(end 117.79 75.52)
@@
 	)
 	(segment
-		(start 171.32 67.77)
-		(end 170.31 68.78)
-		(width 1)
-		(layer "B.Cu")
-		(net "GND")
-	)
-	(segment
 		(start 154.46 75.77)
 		(end 154.46 74.58)
@@
 	)
 	(segment
-		(start 171.105 71.955)
-		(end 172.36 71.955)
-		(width 1)
-		(layer "B.Cu")
-		(net "GND")
-	)
-	(segment
 		(start 117.79 78.79)
 		(end 117.79 77.56)
@@
 		(width 1)
 		(layer "B.Cu")
-		(net "GND")
-	)
-	(segment
-		(start 170.31 68.78)
-		(end 170.31 71.16)
-		(width 1)
-		(layer "B.Cu")
