File: 4ch-spdt-relay-1fan-pcb.kicad_sch (KiCad schematic)
At the start: 45 parts, among them J1 Screw_Terminal_01x03, J2 Conn_01x08_Pin, J3 Screw_Terminal_01x03, J4 Screw_Terminal_01x03, J5 Screw_Terminal_01x03, K1 G5LE-1, K2 G5LE-1, K3 G5LE-1, K4 G5LE-1, Q1 2N3904, Q2 2N3904, Q3 2N3904, Q4 2N3904, Q5 BT136, U5 MOC3021M, U6 PC817

Commit message: Add files via upload
Parts:
- J6, J8: footprint TerminalBlock:TerminalBlock_MaiXu_MX126-5.0-02P_1x02_P5.00mm -> TerminalBlock_Phoenix:TerminalBlock_Phoenix_MKDS-1,5-2-5.08_1x02_P5.08mm_Horizontal
Changed lines of the file:
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@@
 			)
 		)
-		(property "Footprint" "TerminalBlock:TerminalBlock_MaiXu_MX126-5.0-02P_1x02_P5.00mm"
+		(property "Footprint" "TerminalBlock_Phoenix:TerminalBlock_Phoenix_MKDS-1,5-2-5.08_1x02_P5.08mm_Horizontal"
 			(at 104.14 162.5599 0)
 			(hide yes)
@@
 			)
 		)
-		(property "Footprint" "TerminalBlock:TerminalBlock_MaiXu_MX126-5.0-02P_1x02_P5.00mm"
+		(property "Footprint" "TerminalBlock_Phoenix:TerminalBlock_Phoenix_MKDS-1,5-2-5.08_1x02_P5.08mm_Horizontal"
 			(at 62.23 147.3199 0)
 			(hide yes)
